File: PCB+Schematic/Nixie_SevenSegment_Without_IC.kicad_sch (KiCad schematic)
At the start: 27 parts, among them J1 Conn_01x08_Male, U1 WS2811, U2 WS2811, U3 WS2811

Commit message: added resistor values
Parts:
- R10, R8, R9: value R -> 100R
Changed lines of the file:
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@@
       (effects (font (size 1.27 1.27)) (justify left))
     )
-    (property "Value" "R" (id 1) (at 87.63 40.6399 0)
+    (property "Value" "100R" (id 1) (at 87.63 40.6399 0)
       (effects (font (size 1.27 1.27)) (justify left))
     )
@@
       (effects (font (size 1.27 1.27)) (justify left))
     )
-    (property "Value" "R" (id 1) (at 24.13 40.6399 0)
+    (property "Value" "100R" (id 1) (at 24.13 40.6399 0)
       (effects (font (size 1.27 1.27)) (justify left))
     )
@@
       (effects (font (size 1.27 1.27)) (justify left))
     )
-    (property "Value" "R" (id 1) (at 55.88 40.6399 0)
+    (property "Value" "100R" (id 1) (at 55.88 40.6399 0)
       (effects (font (size 1.27 1.27)) (justify left))
     )
@@
     )
     (path "/3c0902bf-745d-4478-b604-bfb41d7626d8"
-      (reference "R8") (unit 1) (value "R") (footprint "Resistor_SMD:R_0805_2012Metric_Pad1.20x1.40mm_HandSolder")
+      (reference "R8") (unit 1) (value "100R") (footprint "Resistor_SMD:R_0805_2012Metric_Pad1.20x1.40mm_HandSolder")
     )
     (path "/91069721-fdb8-46c1-adb2-457fe08c5858"
-      (reference "R9") (unit 1) (value "R") (footprint "Resistor_SMD:R_0805_2012Metric_Pad1.20x1.40mm_HandSolder")
+      (reference "R9") (unit 1) (value "100R") (footprint "Resistor_SMD:R_0805_2012Metric_Pad1.20x1.40mm_HandSolder")
     )
     (path "/2e9c767a-dcdc-4451-b305-337f9b1a904b"
-      (reference "R10") (unit 1) (value "R") (footprint "Resistor_SMD:R_0805_2012Metric_Pad1.20x1.40mm_HandSolder")
+      (reference "R10") (unit 1) (value "100R") (footprint "Resistor_SMD:R_0805_2012Metric_Pad1.20x1.40mm_HandSolder")
     )
     (path "/59b02917-1da6-40a1-9865-daa08474c094"
